File: PCB/new-dev-board/new-dev-board.kicad_pcb (KiCad board)
At the start: 2 copper layers, 185 x 135 mm, 4 parts, among them J1 SIM7600

Commit message: removed power traces. added pwr plane
Parts:
- moved A1 42.8 mm to (100.5, 87.3)
- moved A2 42.8 mm to (118.2, 87.3)
- moved Je1 42.8 mm to (161.3, 133.9)
- moved J1 42.8 mm to (194.2, 50.1)
Routing:
- net /TSC_STM/GND: track 441.3 -> 0.00 mm
- net /TSC_STM/E5V: track 272.0 -> 0.00 mm
- added copper zone on F.Cu, net /TSC_STM/E5V
- removed copper zone on F.Cu, net /TSC_STM/GND
Changed lines of the file:
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@@
   (net 477 "unconnected-(J1-Pin_40-Pad40)")
   (footprint "NUCLEO-F767ZI:SIM7600" (layer "F.Cu")
-    (at 151.4 50.8)
+    (at 194.2 50.1)
     (property "Sheetfile" "new-dev-board.kicad_sch")
     (property "Sheetname" "")
@@
   )
   (footprint "TerminalBlock_Phoenix:TerminalBlock_Phoenix_MKDS-1,5-2-5.08_1x02_P5.08mm_Horizontal" (layer "F.Cu")
-    (at 118.52 134.6)
+    (at 161.32 133.9)
     (descr "Terminal Block Phoenix MKDS-1,5-2-5.08, 2 pins, pitch 5.08mm, size 10.2x9.8mm^2, drill diamater 1.3mm, pad diameter 2.6mm, see http://www.farnell.com/datasheets/100425.pdf, script-generated using https://github.com/pointhi/kicad-footprint-generator/scripts/TerminalBlock_Phoenix")
     (tags "THT Terminal Block Phoenix MKDS-1,5-2-5.08 pitch 5.08mm size 10.2x9.8mm^2 drill 1.3mm pad 2.6mm")
@@
   )
   (footprint "NUCLEO-F767ZI:NUCLEO-F767ZI" (layer "F.Cu")
-    (at 57.7 88.01)
+    (at 100.5 87.31)
     (property "MANUFACTURER" "STMicroelectronics")
     (property "MAXIMUM_PACKAGE_HEIGHT" "N/A")
@@
   )
   (footprint "NUCLEO-F767ZI:NUCLEO-F767ZI" (layer "B.Cu")
-    (at 75.4 88 180)
+    (at 118.2 87.3 180)
     (property "MANUFACTURER" "STMicroelectronics")
     (property "MAXIMUM_PACKAGE_HEIGHT" "N/A")
@@
       (net 384 "Net-(A2B-GND_CN12-PadCN12_20)") (pinfunction "GND_CN12") (pintype "power_in"))
   )
-  (gr_rect (start 20 20) (end 205 155)
+  (gr_rect (start 52.5 19.8) (end 237.5 154.8)
     (stroke (width 0.1) (type default)) (fill none) (layer "Edge.Cuts"))
-  (segment (start 104.61 58.15) (end 99.15 58.15) (width 0.25) (layer "F.Cu") (net 6))
-  (segment (start 28.49 58.16) (end 61.75 24.9) (width 0.25) (layer "F.Cu") (net 6))
-  (segment (start 94.8 44) (end 113.9 24.9) (width 0.25) (layer "F.Cu") (net 6))
-  (segment (start 123.6 28.44) (end 127.14 24.9) (width 0.25) (layer "F.Cu") (net 6))
-  (segment (start 94.8 53.8) (end 94.8 44) (width 0.25) (layer "F.Cu") (net 6))
-  (segment (start 61.75 24.9) (end 113.9 24.9) (width 0.25) (layer "F.Cu") (net 6))
-  (segment (start 99.15 58.15) (end 94.8 53.8) (width 0.25) (layer "F.Cu") (net 6))
-  (segment (start 113.9 24.9) (end 127.14 24.9) (width 0.25) (layer "F.Cu") (net 6))
-  (segment (start 123.6 134.6) (end 123.6 28.44) (width 0.25) (layer "F.Cu") (net 6))
-  (segment (start 114.2 144.4) (end 126.4 144.4) (width 0.25) (layer "F.Cu") (net 74))
-  (segment (start 111.2 141.4) (end 114.2 144.4) (width 0.25) (layer "F.Cu") (net 74))
-  (segment (start 114.2 134.6) (end 111.2 137.6) (width 0.25) (layer "F.Cu") (net 74))
-  (segment (start 131.2 139.6) (end 131.2 33.54) (width 0.25) (layer "F.Cu") (net 74))
-  (segment (start 111.2 137.6) (end 111.2 141.4) (width 0.25) (layer "F.Cu") (net 74))
-  (segment (start 118.52 134.6) (end 114.2 134.6) (width 0.25) (layer "F.Cu") (net 74))
-  (segment (start 126.4 144.4) (end 131.2 139.6) (width 0.25) (layer "F.Cu") (net 74))
-  (segment (start 131.2 33.54) (end 137.3 27.44) (width 0.25) (layer "F.Cu") (net 74))
-  (segment (start 102.6 72.86) (end 99.53 75.93) (width 0.25) (layer "B.Cu") (net 74))
-  (segment (start 118.52 134.6) (end 118.52 137.88) (width 0.25) (layer "B.Cu") (net 74))
-  (segment (start 50.618507 150.5) (end 31 130.881493) (width 0.25) (layer "B.Cu") (net 74))
-  (segment (start 118.52 134.6) (end 118.52 47.6) (width 0.25) (layer "B.Cu") (net 74))
-  (segment (start 102.6 49.8) (end 102.6 72.86) (width 0.25) (layer "B.Cu") (net 74))
-  (segment (start 31 81.05) (end 33.57 78.48) (width 0.25) (layer "B.Cu") (net 74))
-  (segment (start 118.52 47.32) (end 116.4 45.2) (width 0.25) (layer "B.Cu") (net 74))
-  (segment (start 118.52 47.6) (end 118.52 47.32) (width 0.25) (layer "B.Cu") (net 74))
-  (segment (start 105.9 150.5) (end 50.618507 150.5) (width 0.25) (layer "B.Cu") (net 74))
-  (segment (start 31 130.881493) (end 31 81.05) (width 0.25) (layer "B.Cu") (net 74))
-  (segment (start 118.52 137.88) (end 105.9 150.5) (width 0.25) (layer "B.Cu") (net 74))
-  (segment (start 107.2 45.2) (end 102.6 49.8) (width 0.25) (layer "B.Cu") (net 74))
-  (segment (start 116.4 45.2) (end 107.2 45.2) (width 0.25) (layer "B.Cu") (net 74))
-  (segment (start 66.05 107.75) (end 50.55 107.75) (width 0.25) (layer "F.Cu") (net 124))
-  (segment (start 50.55 107.75) (end 49.8 107) (width 0.25) (layer "F.Cu") (net 124))
-  (segment (start 80.38 102.79) (end 71.01 102.79) (width 0.25) (layer "F.Cu") (net 124))
-  (segment (start 81.83 101.34) (end 80.38 102.79) (width 0.25) (layer "F.Cu") (net 124))
-  (segment (start 71.01 102.79) (end 66.05 107.75) (width 0.25) (layer "F.Cu") (net 124))
-  (segment (start 49.8 107) (end 49.8 105.34) (width 0.25) (layer "F.Cu") (net 124))
-  (segment (start 49.8 105.34) (end 51.27 103.87) (width 0.25) (layer "F.Cu") (net 124))
-  (segment (start 180.2 24.6) (end 177.2 21.6) (width 0.25) (layer "F.Cu") (net 341))
-  (segment (start 180.2 31) (end 180.2 24.6) (width 0.25) (layer "F.Cu") (net 341))
-  (segment (start 130.1 147.3) (end 137.4 140) (width 0.25) (layer "F.Cu") (net 341))
-  (segment (start 177.2 21.6) (end 140.6 21.6) (width 0.25) (layer "F.Cu") (net 341))
-  (segment (start 49 127.2) (end 69.1 147.3) (width 0.25) (layer "F.Cu") (net 341))
-  (segment (start 178 33.2) (end 180.2 31) (width 0.25) (layer "F.Cu") (net 341))
-  (segment (start 137.4 36.6) (end 140.8 33.2) (width 0.25) (layer "F.Cu") (net 341))
-  (segment (start 137.4 140) (end 137.4 36.6) (width 0.25) (layer "F.Cu") (net 341))
-  (segment (start 51.27 96.25) (end 49 98.52) (width 0.25) (layer "F.Cu") (net 341))
-  (segment (start 140.8 33.2) (end 178 33.2) (width 0.25) (layer "F.Cu") (net 341))
-  (segment (start 140.6 21.6) (end 137.3 24.9) (width 0.25) (layer "F.Cu") (net 341))
-  (segment (start 69.1 147.3) (end 130.1 147.3) (width 0.25) (layer "F.Cu") (net 341))
-  (segment (start 49 98.52) (end 49 127.2) (width 0.25) (layer "F.Cu") (net 341))
-  (segment (start 48.8 49.4) (end 48.8 96.32) (width 0.25) (layer "B.Cu") (net 343))
-  (segment (start 48.8 96.32) (end 51.27 98.79) (width 0.25) (layer "B.Cu") (net 343))
-  (segment (start 131.86 22) (end 76.2 22) (width 0.25) (layer "B.Cu") (net 343))
-  (segment (start 76.2 22) (end 48.8 49.4) (width 0.25) (layer "B.Cu") (net 343))
-  (segment (start 134.76 24.9) (end 131.86 22) (width 0.25) (layer "B.Cu") (net 343))
-  (zone (net 74) (net_name "/TSC_STM/GND") (layers "F&B.Cu") (hatch edge 0.5)
+  (segment (start 123.37 101.9) (end 114 101.9) (width 0.25) (layer "F.Cu") (net 124))
+  (segment (start 92.6 106.3) (end 92.6 104.64) (width 0.25) (layer "F.Cu") (net 124))
+  (segment (start 124.63 100.64) (end 123.37 101.9) (width 0.25) (layer "F.Cu") (net 124))
+  (segment (start 108.95 106.95) (end 93.25 106.95) (width 0.25) (layer "F.Cu") (net 124))
+  (segment (start 93.25 106.95) (end 92.6 106.3) (width 0.25) (layer "F.Cu") (net 124))
+  (segment (start 92.6 104.64) (end 94.07 103.17) (width 0.25) (layer "F.Cu") (net 124))
+  (segment (start 114 101.9) (end 108.95 106.95) (width 0.25) (layer "F.Cu") (net 124))
+  (segment (start 223 23.9) (end 220 20.9) (width 0.25) (layer "F.Cu") (net 341))
+  (segment (start 223 30.3) (end 223 23.9) (width 0.25) (layer "F.Cu") (net 341))
+  (segment (start 172.9 146.6) (end 180.2 139.3) (width 0.25) (layer "F.Cu") (net 341))
+  (segment (start 220 20.9) (end 183.4 20.9) (width 0.25) (layer "F.Cu") (net 341))
+  (segment (start 91.8 126.5) (end 111.9 146.6) (width 0.25) (layer "F.Cu") (net 341))
+  (segment (start 220.8 32.5) (end 223 30.3) (width 0.25) (layer "F.Cu") (net 341))
+  (segment (start 180.2 35.9) (end 183.6 32.5) (width 0.25) (layer "F.Cu") (net 341))
+  (segment (start 180.2 139.3) (end 180.2 35.9) (width 0.25) (layer "F.Cu") (net 341))
+  (segment (start 94.07 95.55) (end 91.8 97.82) (width 0.25) (layer "F.Cu") (net 341))
+  (segment (start 183.6 32.5) (end 220.8 32.5) (width 0.25) (layer "F.Cu") (net 341))
+  (segment (start 183.4 20.9) (end 180.1 24.2) (width 0.25) (layer "F.Cu") (net 341))
+  (segment (start 111.9 146.6) (end 172.9 146.6) (width 0.25) (layer "F.Cu") (net 341))
+  (segment (start 91.8 97.82) (end 91.8 126.5) (width 0.25) (layer "F.Cu") (net 341))
+  (segment (start 91.6 48.7) (end 91.6 95.62) (width 0.25) (layer "B.Cu") (net 343))
+  (segment (start 91.6 95.62) (end 94.07 98.09) (width 0.25) (layer "B.Cu") (net 343))
+  (segment (start 174.66 21.3) (end 119 21.3) (width 0.25) (layer "B.Cu") (net 343))
+  (segment (start 119 21.3) (end 91.6 48.7) (width 0.25) (layer "B.Cu") (net 343))
+  (segment (start 177.56 24.2) (end 174.66 21.3) (width 0.25) (layer "B.Cu") (net 343))
+  (zone (net 6) (net_name "/TSC_STM/E5V") (layer "F.Cu") (hatch edge 0.5)
     (connect_pads (clearance 0.5))
     (min_thickness 0.25) (filled_areas_thickness no)
@@
     (polygon
       (pts
-        (xy 17.65 17.05)
-        (xy 209.35 16.1)
-        (xy 210.8 160.05)
-        (xy 15.5 158.7)
+        (xy -5.35 -9.65)
+        (xy 310.1 -10.45)
+        (xy 311.1 225.6)
+        (xy -12.3 224.6)
       )
     )
+  )
+  (zone (net 74) (net_name "/TSC_STM/GND") (layer "B.Cu") (hatch edge 0.5)
+    (priority 1)
+    (connect_pads (clearance 0.5))
+    (min_thickness 0.25) (filled_areas_thickness no)
+    (fill yes (thermal_gap 0.5) (thermal_bridge_width 0.5))
+    (polygon
+      (pts
+        (xy -14.55 -22.5)
+        (xy 321.7 -21.9)
+        (xy 323.5 239.6)
+        (xy -27.6 243.55)
+      )
+    )
