File: PCB/dev-boards/tsc_side.kicad_sch (KiCad schematic)
At the start: 1 part, among them U3 NUCLEO-F429ZI

Commit message: PCB board updates
Signed-off-by: Andrew Balmos <abalmos@purdue.edu>
Connections:
- net D_TX: now also U3.CN10_18 (D42/TIMER_A_PWM1N); no longer U3.CN12_40 (PE8)
Changed lines of the file:
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@@
-    (stroke (width 0) (type default))
-  )
-  (wire (pts (xy 55.88 59.055) (xy 60.96 59.055))
     (stroke (width 0) (type default))
   )
@@
     (stroke (width 0) (type default))
   )
+  (wire (pts (xy 193.04 136.525) (xy 196.215 136.525))
+    (stroke (width 0) (type default))
+  )
   (wire (pts (xy 58.42 127.635) (xy 58.42 128.905))
     (stroke (width 0) (type default))
@@
     (stroke (width 0) (type default))
   )
-  (hierarchical_label "D_TX" (shape output) (at 60.96 59.055 0) (fields_autoplaced)
-    (effects (font (size 1.27 1.27)) (justify left))
+  (hierarchical_label "D_TX" (shape output) (at 193.04 136.525 180) (fields_autoplaced)
+    (effects (font (size 1.27 1.27)) (justify right))
   )
   (symbol (lib_id "Nucleo-144:NUCLEO-F429ZI") (at 38.1 76.835 0) (unit 2)

Commit message: Update PCB for JLCPCB
Signed-off-by: Andrew Balmos <abalmos@purdue.edu>
Parts:
- U3: footprint MODULE_NUCLEO-F429ZI -> Local footprints:MODULE_NUCLEO-F429ZI
Changed lines of the file:
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@@
   (symbol (lib_id "Nucleo-144:NUCLEO-F429ZI") (at 38.1 76.835 0) (unit 2)
     (in_bom yes) (on_board yes) (dnp no)
-    (property "Reference" "U3" (at 161.29 15.875 0)
+    (property "Reference" "U3" (at 38.1 17.272 0)
       (effects (font (size 1.27 1.27)))
     )
@@
       (effects (font (size 1.27 1.27)))
     )
-    (property "Footprint" "MODULE_NUCLEO-F429ZI" (at 38.1 76.835 0)
+    (property "Footprint" "Local footprints:MODULE_NUCLEO-F429ZI" (at 38.1 76.835 0)
       (effects (font (size 1.27 1.27)) (justify bottom) hide)
     )
@@
       (effects (font (size 1.27 1.27)) hide)
     )
-    (property "Footprint" "MODULE_NUCLEO-F429ZI" (at 223.52 52.07 0)
+    (property "Footprint" "Local footprints:MODULE_NUCLEO-F429ZI" (at 223.52 52.07 0)
       (effects (font (size 1.27 1.27)) (justify bottom) hide)
     )
@@
       (effects (font (size 1.27 1.27)))
     )
-    (property "Footprint" "MODULE_NUCLEO-F429ZI" (at 229.235 121.285 0)
+    (property "Footprint" "Local footprints:MODULE_NUCLEO-F429ZI" (at 229.235 121.285 0)
       (effects (font (size 1.27 1.27)) (justify bottom) hide)
     )
@@
       (effects (font (size 1.27 1.27)))
     )
-    (property "Footprint" "MODULE_NUCLEO-F429ZI" (at 86.36 76.835 0)
+    (property "Footprint" "Local footprints:MODULE_NUCLEO-F429ZI" (at 86.36 76.835 0)
       (effects (font (size 1.27 1.27)) (justify bottom) hide)
     )
@@
       (effects (font (size 1.27 1.27)))
     )
-    (property "Footprint" "MODULE_NUCLEO-F429ZI" (at 147.955 121.285 0)
+    (property "Footprint" "Local footprints:MODULE_NUCLEO-F429ZI" (at 147.955 121.285 0)
       (effects (font (size 1.27 1.27)) (justify bottom) hide)
     )
@@
       (effects (font (size 1.27 1.27)))
     )
-    (property "Footprint" "MODULE_NUCLEO-F429ZI" (at 144.145 52.07 0)
-      (effects (font (size 1.27 1.27)) (justify bottom) hide)
-    )
+    (property "Footprint" "Local footprints:MODULE_NUCLEO-F429ZI" (at 144.145 52.07 0)
+      (effects (font (size 1.27 1.27)) (justify bottom) hide)
+    )
