File: PCB/dev-boards/dev-boards.kicad_sch (KiCad schematic)
At the start: 2 parts, among them J1 Screw_Terminal_01x02, J2 SIM7600 Dev Board

Commit message: PCB board updates
Signed-off-by: Andrew Balmos <abalmos@purdue.edu>
Parts:
- J1: value Screw_Terminal_01x02 -> 5V Input
- J2: value SIM7600 Dev Board -> SIM7600 Cell Header; symbol Connector_Generic:Conn_02x20_Counter_Clockwise -> Connector_Generic:Conn_02x20_Odd_Even
Connections:
- net +5V: now also J2.2 (Pin_2), J2.4 (Pin_4); no longer J2.39 (Pin_39), J2.40 (Pin_40)
- net GND: now also J2.14 (Pin_14), J2.25 (Pin_25), J2.30 (Pin_30), J2.39 (Pin_39), J2.6 (Pin_6), J2.9 (Pin_9); no longer J2.13 (Pin_13), J2.24 (Pin_24), J2.26 (Pin_26), J2.31 (Pin_31), J2.38 (Pin_38), J2.5 (Pin_5)
- net M_RX_TX: now reaches J2.10 (Pin_10)
- net M_TX_RX: now reaches J2.8 (Pin_8)
Other:
- sheet WorldSide Sheet ports: added M_RX, M_TX; removed none
- note added: "Cell Modem"
- note added: "Data Diode"
- note added: "Power"
- moved on the sheet: J1, J2

Commit message: Update PCB for JLCPCB
Signed-off-by: Andrew Balmos <abalmos@purdue.edu>
Parts:
- added H1, H2: MountingHole, MountingHole:MountingHole_4.3mm_M4, symbol Mechanical:MountingHole
- added N1: Housing, Local footprints:oats_logo, symbol Mechanical:Housing
Changed lines of the file:
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@@
+    )
+  )
+  (symbol (lib_id "Mechanical:MountingHole") (at 88.392 177.292 0) (unit 1)
+    (in_bom yes) (on_board yes) (dnp no) (fields_autoplaced)
+    (property "Reference" "H2" (at 91.948 176.657 0)
+      (effects (font (size 1.27 1.27)) (justify left))
+    )
+    (property "Value" "MountingHole" (at 91.948 179.197 0)
+      (effects (font (size 1.27 1.27)) (justify left))
+    )
+    (property "Footprint" "MountingHole:MountingHole_4.3mm_M4" (at 88.392 177.292 0)
+      (effects (font (size 1.27 1.27)) hide)
+    )
+    (property "Datasheet" "~" (at 88.392 177.292 0)
+      (effects (font (size 1.27 1.27)) hide)
+    )
+    (instances
+      (project "dev-boards"
+        (path "/e2f9bcb9-b304-4d0a-965b-237a65fc186b"
+          (reference "H2") (unit 1)
+        )
+      )
     )
   )
@@
     )
   )
+  (symbol (lib_id "Mechanical:Housing") (at 40.386 177.038 0) (unit 1)
+    (in_bom yes) (on_board yes) (dnp no) (fields_autoplaced)
+    (property "Reference" "N1" (at 46.482 176.7205 0)
+      (effects (font (size 1.27 1.27)) (justify left))
+    )
+    (property "Value" "Housing" (at 46.482 179.2605 0)
+      (effects (font (size 1.27 1.27)) (justify left))
+    )
+    (property "Footprint" "Local footprints:oats_logo" (at 41.656 175.768 0)
+      (effects (font (size 1.27 1.27)) hide)
+    )
+    (property "Datasheet" "~" (at 41.656 175.768 0)
+      (effects (font (size 1.27 1.27)) hide)
+    )
+    (instances
+      (project "dev-boards"
+        (path "/e2f9bcb9-b304-4d0a-965b-237a65fc186b"
+          (reference "N1") (unit 1)
+        )
+      )
+    )
+  )
   (symbol (lib_id "power:+5V") (at 47.752 84.582 0) (unit 1)
     (in_bom yes) (on_board yes) (dnp no) (fields_autoplaced)
@@
         )
       )
+    )
+  )
+  (symbol (lib_id "Mechanical:MountingHole") (at 65.024 176.784 0) (unit 1)
+    (in_bom yes) (on_board yes) (dnp no) (fields_autoplaced)
+    (property "Reference" "H1" (at 68.58 176.149 0)
+      (effects (font (size 1.27 1.27)) (justify left))
+    )
+    (property "Value" "MountingHole" (at 68.58 178.689 0)
+      (effects (font (size 1.27 1.27)) (justify left))
+    )
+    (property "Footprint" "MountingHole:MountingHole_4.3mm_M4" (at 65.024 176.784 0)
+      (effects (font (size 1.27 1.27)) hide)
+    )
+    (property "Datasheet" "~" (at 65.024 176.784 0)
+      (effects (font (size 1.27 1.27)) hide)
+    )
+    (instances
+      (project "dev-boards"
+        (path "/e2f9bcb9-b304-4d0a-965b-237a65fc186b"
+          (reference "H1") (unit 1)
+        )
+      )

Commit message: PCB: Edits for 3d box
Signed-off-by: Andrew Balmos <abalmos@purdue.edu>
Parts:
- added H3: MountingHole, MountingHole:MountingHole_3.5mm, symbol Mechanical:MountingHole
- H1, H2: footprint MountingHole:MountingHole_4.3mm_M4 -> MountingHole:MountingHole_3.5mm
Changed lines of the file:
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@@
+    )
+  )
+  (symbol (lib_id "Mechanical:MountingHole") (at 65.024 185.674 0) (unit 1)
+    (in_bom yes) (on_board yes) (dnp no) (fields_autoplaced)
+    (property "Reference" "H3" (at 68.58 185.039 0)
+      (effects (font (size 1.27 1.27)) (justify left))
+    )
+    (property "Value" "MountingHole" (at 68.58 187.579 0)
+      (effects (font (size 1.27 1.27)) (justify left))
+    )
+    (property "Footprint" "MountingHole:MountingHole_3.5mm" (at 65.024 185.674 0)
+      (effects (font (size 1.27 1.27)) hide)
+    )
+    (property "Datasheet" "~" (at 65.024 185.674 0)
+      (effects (font (size 1.27 1.27)) hide)
+    )
+    (instances
+      (project "dev-boards"
+        (path "/e2f9bcb9-b304-4d0a-965b-237a65fc186b"
+          (reference "H3") (unit 1)
+        )
+      )
     )
   )
@@
       (effects (font (size 1.27 1.27)) (justify left))
     )
-    (property "Footprint" "MountingHole:MountingHole_4.3mm_M4" (at 88.392 177.292 0)
+    (property "Footprint" "MountingHole:MountingHole_3.5mm" (at 88.392 177.292 0)
       (effects (font (size 1.27 1.27)) hide)
     )
@@
       (effects (font (size 1.27 1.27)) (justify left))
     )
-    (property "Footprint" "MountingHole:MountingHole_4.3mm_M4" (at 65.024 176.784 0)
-      (effects (font (size 1.27 1.27)) hide)
-    )
+    (property "Footprint" "MountingHole:MountingHole_3.5mm" (at 65.024 176.784 0)
+      (effects (font (size 1.27 1.27)) hide)
+    )
